Commit message: URDF Python and related changes to URDF Tools
git-svn-id: https://wu-ros-pkg.svn.sourceforge.net/svnroot/wu-ros-pkg/stacks/urdf_tools/trunk@47 8be2bc32-520c-440a-ab74-22c12e9655a8

File: urdf_tutorial/08-macroed.urdf.xacro (robot description, xacro)
@@ -58,5 +58,5 @@
 			<origin xyz="0 ${baselen*reflect/3} -${wheeldiam/2+.05}" rpy="0 ${pi/2} 0"/>
       			<limit effort="100" velocity="100" />
-			<joint_properties damping="0.0" friction="0.0" />
+			<dynamics damping="0.0" friction="0.0" />
 		</joint>
 	</xacro:macro>
